Commit message: 【feat】添加天机696型号机械臂URDF文件并适配

File: e1_pro_full/urdf/E1-PRO_EVT2.0_V12_260730.urdf (robot description, URDF)
Before this commit: robot E1-PRO_EVT2.0_V9_260714, 15 links, 14 joints
Links:
- removed link boxs02_link
- removed link left_dianchi_link
- removed link paltform_link
- removed link right_dianchi_link
- removed link zhijian_link
- added link CTU_link, mass 7.2262; collision mesh filename=package://E1-PRO_EVT2.0_V12_260730/meshes/CTU_link.STL; visual mesh filename=package://E1-PRO_EVT2.0_V12_260730/meshes/CTU_link.STL
- added link box02_link, mass 10.895; collision mesh filename=package://E1-PRO_EVT2.0_V12_260730/meshes/box02_link.STL; visual mesh filename=package://E1-PRO_EVT2.0_V12_260730/meshes/box02_link.STL
- added link end_effector_link, mass 0.27303; collision mesh filename=package://E1-PRO_EVT2.0_V12_260730/meshes/end_effector_link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; visual mesh filename=package://E1-PRO_EVT2.0_V12_260730/meshes/end_effector_link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
- added link platform_link, mass 34.753; collision mesh filename=package://E1-PRO_EVT2.0_V12_260730/meshes/platform_link.STL; visual mesh filename=package://E1-PRO_EVT2.0_V12_260730/meshes/platform_link.STL
- link Link1_L: mass 0.81851 -> 1.9705; geometry collision mesh filename=package://E1-PRO_EVT2.0_V12_260730/meshes/Link1_L.STL; visual mesh filename=package://E1-PRO_EVT2.0_V12_260730/meshes/Link1_L.STL
- link Link2_L: mass 1.1465 -> 2.24398; geometry collision mesh filename=package://E1-PRO_EVT2.0_V12_260730/meshes/Link2_L.STL; visual mesh filename=package://E1-PRO_EVT2.0_V12_260730/meshes/Link2_L.STL
- link Link3_L: mass 1.859 -> 1.9242; geometry collision mesh filename=package://E1-PRO_EVT2.0_V12_260730/meshes/Link3_L.STL; visual mesh filename=package://E1-PRO_EVT2.0_V12_260730/meshes/Link3_L.STL
- link Link4_L: mass 0.80083 -> 1.6085; geometry collision mesh filename=package://E1-PRO_EVT2.0_V12_260730/meshes/Link4_L.STL; visual mesh filename=package://E1-PRO_EVT2.0_V12_260730/meshes/Link4_L.STL
- link Link5_L: mass 1.6879 -> 2.0883; geometry collision mesh filename=package://E1-PRO_EVT2.0_V12_260730/meshes/Link5_L.STL; visual mesh filename=package://E1-PRO_EVT2.0_V12_260730/meshes/Link5_L.STL
- link Link6_L: mass 0.28617 -> 0.72496; geometry collision mesh filename=package://E1-PRO_EVT2.0_V12_260730/meshes/Link6_L.STL; visual mesh filename=package://E1-PRO_EVT2.0_V12_260730/meshes/Link6_L.STL
- link Link7_L: mass 0.33604 -> 0.68606; geometry collision mesh filename=package://E1-PRO_EVT2.0_V12_260730/meshes/Link7_L.STL; visual mesh filename=package://E1-PRO_EVT2.0_V12_260730/meshes/Link7_L.STL
- link arm_base_link: mass 0.59585 -> 4.7258; geometry collision mesh filename=package://E1-PRO_EVT2.0_V12_260730/meshes/arm_base_link.STL; visual mesh filename=package://E1-PRO_EVT2.0_V12_260730/meshes/arm_base_link.STL
- link base_link: mass 32.049 -> 472.28; geometry collision mesh filename=package://E1-PRO_EVT2.0_V12_260730/meshes/base_link.STL; visual mesh filename=package://E1-PRO_EVT2.0_V12_260730/meshes/base_link.STL
- link box01_link: mass 24.317 -> 8.32; geometry collision mesh filename=package://E1-PRO_EVT2.0_V12_260730/meshes/box01_link.STL; visual mesh filename=package://E1-PRO_EVT2.0_V12_260730/meshes/box01_link.STL
Joints:
- removed joint Joint1_J
- removed joint Joint2_J
- removed joint Joint3_J
- removed joint Joint4_J
- removed joint Joint5_J
- removed joint Joint6_J
- removed joint Joint7_J
- removed joint boxs02_joint
- removed joint left_dainchi_joint
- removed joint right_dianchi_joint
- removed joint zhijian_joint
- added joint CTU_joint: type revolute, parent platform_link, child CTU_link, origin xyz=0.45457 0 1.1259 rpy=0 0 0, axis 0 0 1, limit lower=-3.1416 upper=3.1416 effort=0 velocity=0
- added joint Joint1_L: type revolute, parent arm_base_link, child Link1_L, origin xyz=0 0 0.1745 rpy=0 0 0, axis 0 0 1, limit lower=-3.1067 upper=3.1067 effort=108 velocity=3.1416
- added joint Joint2_L: type revolute, parent Link1_L, child Link2_L, origin xyz=0 0 0 rpy=1.5708 0 0, axis 0 0 1, limit lower=-2.0944 upper=2.0944 effort=108 velocity=3.1416
- added joint Joint3_L: type revolute, parent Link2_L, child Link3_L, origin xyz=0 0.287 0 rpy=-1.5708 0 0, axis 0 0 1, limit lower=-3.1067 upper=3.1067 effort=66 velocity=3.1416
- added joint Joint4_L: type revolute, parent Link3_L, child Link4_L, origin xyz=0.018 0 0 rpy=-1.5708 0 3.1416, axis 0 0 1, limit lower=-2.5307 upper=1.0472 effort=66 velocity=3.1416
- added joint Joint5_L: type revolute, parent Link4_L, child Link5_L, origin xyz=0.018 -0.314 0 rpy=-1.5708 0 3.1416, axis 0 0 1, limit lower=-3.1067 upper=3.1067 effort=18 velocity=3.1416
- added joint Joint6_L: type revolute, parent Link5_L, child Link6_L, origin xyz=0 0 0 rpy=1.5708 -1.5708 0, axis 0 0 1, limit lower=-1.0472 upper=1.0472 effort=18 velocity=3.1416
- added joint Joint7_L: type revolute, parent Link6_L, child Link7_L, origin xyz=0 0 0 rpy=1.5708 -1.5708 0, axis 0 0 1, limit lower=-1.5708 upper=1.5708 effort=18 velocity=3.1416
- added joint box02_joint: type fixed, parent base_link, child box02_link, origin xyz=-0.25162 0.0004972 1.3028 rpy=0 0 0, axis 0 0 0
- added joint end_effector_joint: type fixed, parent Link7_L, child end_effector_link, origin xyz=-0.0083277 -0.17809 0 rpy=1.5708 1.5708 0, axis 0 0 0
- joint arm_base_joint: origin xyz=0.51352 -0.031 0.31 rpy=0 0 0 -> xyz=0.1145 0.2905 1.5345 rpy=0 0 -1.5707963; parent paltform_link -> platform_link
- joint box01_joint: axis 0 1 0 -> 0 0 0; limit lower=-0.7 upper=0.7 effort=0 velocity=0 -> (none); origin xyz=0.14402 -0.031 0.31 rpy=0 0 0 -> xyz=-0.12707 0.00066942 0.1791 rpy=0 0 0; parent paltform_link -> CTU_link; type prismatic -> fixed
- joint platform_joint: child paltform_link -> platform_link; limit lower=-0.1 upper=0.5 effort=0 velocity=0 -> lower=-1 upper=1 effort=0 velocity=0
